File: kicad/file5A71BCB7.sch (KiCad schematic (older format))
At the start: 56 parts, among them J1 GS3, J14 Conn_01x03, J2 Conn_01x05, J3 GS2, J4 GS3, SW1 SW_Push, U1 MAX1658ESA, U2 STM32F102RBTx, Y1 8MHZ

Commit message: added some footprints
Parts:
- U2: footprint LQFP64 -> Housings_QFP:LQFP-64_10x10mm_Pitch0.5mm
Changed lines of the file:
@@
 F 0 "U2" H 4500 5075 50  0000 L BNN
 F 1 "STM32F102RBTx" H 7900 5075 50  0000 R BNN
-F 2 "LQFP64" H 7900 5025 50  0001 R TNN
+F 2 "Housings_QFP:LQFP-64_10x10mm_Pitch0.5mm" H 7900 5025 50  0001 R TNN
 F 3 "" H 6200 3150 50  0001 C CNN
 	1    6200 3150
