File: kicad/file5A71BCC7.sch (KiCad schematic (older format))
At the start: 80 parts, among them J10 Conn_01x01, J11 Conn_01x01, J5 Conn_01x04, J6 Conn_01x01, J7 Conn_01x01, J8 USB_B_Micro, J9 Conn_01x01, Q1 FDMC8651, Q2 FDMC8651, Q3 FDMC8651, Q4 FDMC8651, Q5 IRF7324, Q6 FDMC8651, Q7 FDMC8651, U3 LTC4156, U4 ACS711xLCTR-12AB, U5 ACS711xLCTR-12AB, U6 LTC3119, U7 MAX1709, U8 LM5050, U9 LM5050

Commit message: added some footprints
Parts:
- J8: footprint (none) -> Connectors_USB:USB_Micro-B_Molex_47346-0001
- U8, U9: footprint (none) -> TO_SOT_Packages_SMD:SOT-23-6
Changed lines of the file:
@@
 F 0 "J8" H 3800 7600 50  0000 L CNN
 F 1 "USB_B_Micro" H 3800 7500 50  0000 L CNN
-F 2 "" H 4150 7100 50  0001 C CNN
+F 2 "Connectors_USB:USB_Micro-B_Molex_47346-0001" H 4150 7100 50  0001 C CNN
 F 3 "" H 4150 7100 50  0001 C CNN
 	1    4000 7150
@@
 	2100 2550 3950 2550
 Wire Notes Line
-	3950 2550 3950 3700
-Wire Notes Line
 	3950 3700 550  3700
 Wire Notes Line
@@
 F 0 "U9" H 9600 1450 43  0000 C CNN
 F 1 "LM5050" H 9150 1450 43  0000 C CNN
-F 2 "" H 11300 1900 43  0001 C CNN
+F 2 "TO_SOT_Packages_SMD:SOT-23-6" H 11300 1900 43  0001 C CNN
 F 3 "" H 11300 1900 43  0001 C CNN
 	1    9350 1750
@@
 F 0 "U8" H 9550 3350 43  0000 C CNN
 F 1 "LM5050" H 9100 3350 43  0000 C CNN
-F 2 "" H 11250 3800 43  0001 C CNN
+F 2 "TO_SOT_Packages_SMD:SOT-23-6" H 11250 3800 43  0001 C CNN
 F 3 "" H 11250 3800 43  0001 C CNN
 	1    9300 3650
@@
 	5850 6300 6400 6300
 Connection ~ 5850 6300
+Wire Notes Line
+	3950 2550 3950 3700
 $EndSCHEMATC
