File: kicad/file5AAECC8A.sch (KiCad schematic (older format))
At the start: 8 parts, among them J12 USB_A, J13 USB_A, U10 TPS2514A, U11 TPS2514A, U12 TPS2561

Commit message: added some footprints
Parts:
- J12, J13: footprint (none) -> Connectors:USB_A
Changed lines of the file:
@@
 F 0 "J12" H 1150 2050 50  0000 L CNN
 F 1 "USB_A" H 1150 1950 50  0000 L CNN
-F 2 "" H 1500 1550 50  0001 C CNN
+F 2 "Connectors:USB_A" H 1500 1550 50  0001 C CNN
 F 3 "" H 1500 1550 50  0001 C CNN
 	1    1350 1600
@@
 F 0 "J13" H 1150 3200 50  0000 L CNN
 F 1 "USB_A" H 1150 3100 50  0000 L CNN
-F 2 "" H 1500 2700 50  0001 C CNN
+F 2 "Connectors:USB_A" H 1500 2700 50  0001 C CNN
 F 3 "" H 1500 2700 50  0001 C CNN
 	1    1350 2750
